File: Projects/Active label/active label/active label.kicad_pcb (KiCad board)
At the start: 4 copper layers, 170 x 35 mm, 63 parts, among them J1 SFV24R-4STE1HLF, J2 USB4105-GF-A, J3 SM02B-SRSS-TB LFSN, J4 SM02B-SRSS-TB LFSN, J6 SM04B-SRSS-TB, J7 SM04B-SRSS-TB, J8 SM03B-SRSS-TBLFSN, Q1 SI1308EDL, SW1 SW_MEC_5E, SW2 SW_MEC_5E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

Commit message: Layout under way
Parts:
- moved C10 32.8 mm to (140.6, 125.2)
- moved C17 26.8 mm to (141.8, 141.4), turned to -90 degrees
- moved C19 19.1 mm to (149.3, 145.0)
- moved C21 17.1 mm to (154.8, 137.9)
- moved C18 13.5 mm to (154.8, 140.1)
- moved C11 13.3 mm to (161.3, 142.5)
- moved D2 13.2 mm to (140.6, 127.5)
- moved C20 11.6 mm to (154.7, 142.3)
- moved L1 10.9 mm to (147.3, 138.9), turned to 90 degrees
- moved R5 10.5 mm to (161.4, 140.1), turned to 180 degrees
- moved R6 10.3 mm to (168.4, 135.6), turned to 180 degrees
- moved C12 9.69 mm to (139.2, 137.3), turned to -90 degrees
- moved D4 9.58 mm to (141.5, 135.7), turned to -90 degrees
- moved D3 8.52 mm to (140.6, 129.9)
- moved Q1 7.21 mm to (162.9, 136.4), turned to -90 degrees
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Connections:
- J2 pad A8: Net-(J2-SBU1) -> unconnected-(J2-SBU1-PadA8)
- J2 pad B4-A9: unconnected-(J2-VBUS-PadB4-A9) -> VUSB
- J2 pad B5: unconnected-(J2-CC2-PadB5) -> Net-(J2-CC2)
- R2 pad 1: GND -> Net-(J2-CC2)
- R2 pad 2: Net-(J2-SBU1) -> GND
Routing:
- net Net-(D1-Pad1): track 0.00 -> 111.5 mm
- net VBAT_SENSE: track 0.00 -> 106.2 mm
- net VUSB_SENSE: track 0.00 -> 90.5 mm, vias 0 -> 2
- net USBD+: track 0.00 -> 79.0 mm, vias 0 -> 2
- net USBD-: track 0.00 -> 76.8 mm, vias 0 -> 2
- net SWITCH_L: track 0.00 -> 61.4 mm, vias 0 -> 2
- net SDA1: track 0.00 -> 45.3 mm, vias 0 -> 2
- net SDA0: track 0.00 -> 44.9 mm, vias 0 -> 2
- net SCL0: track 0.00 -> 42.0 mm, vias 0 -> 2
- net GND: track 0.00 -> 40.7 mm, vias 0 -> 26
- net SCL1: track 0.00 -> 36.8 mm
- net Net-(Q1-D): track 0.00 -> 36.3 mm, vias 0 -> 5
- net VUSB: track 0.00 -> 22.7 mm, vias 0 -> 3
- net VSL: track 0.00 -> 19.0 mm, vias 0 -> 2
- net +3V3: track 0.00 -> 18.1 mm, vias 0 -> 11
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- added copper zone on In2.Cu, net +3V3
- added copper zone on In1.Cu, net GND
