File: Projects/Active label/active label/active label.kicad_sch (KiCad schematic)
At the start: 63 parts, among them J1 SFV24R-4STE1HLF, J2 USB4105-GF-A, J3 SM02B-SRSS-TB LFSN, J4 SM02B-SRSS-TB LFSN, J6 SM04B-SRSS-TB, J7 SM04B-SRSS-TB, J8 SM03B-SRSS-TBLFSN, Q1 SI1308EDL, SW1 SW_MEC_5E, SW2 SW_MEC_5E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

Commit message: Board layout complete
Connections:
- net at C22.1, U1.9 (IO16): now also Y1.4; no longer Y1.2
Changed lines of the file:
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@@
 			)
 		)
-		(pin "2"
+		(property "FirecoPN" ""
+			(at 66.04 96.52 0)
+			(effects
+				(font
+					(size 1.27 1.27)
+				)
+			)
+		)
+		(property "Manufacturer" ""
+			(at 66.04 96.52 0)
+			(effects
+				(font
+					(size 1.27 1.27)
+				)
+				(hide yes)
+			)
+		)
+		(pin "4"
 		)
 		(pin "1"
